Commit message: 🔧 golf cart model 🤖

File: src/driver/urdf/robot.urdf (robot description, URDF)
Before this commit: robot Alan-v2, 1 links, 0 joints
Links:
- added link steering_subassem; visual mesh filename=package://driver/meshes/steering_subassem.stl.stl scale=0.001 0.001 0.001
- added link steering_wheel_fl; visual mesh filename=package://driver/meshes/wheel_subassem.stl.stl scale=0.001 0.001 0.001
- added link steering_wheel_fr; visual mesh filename=package://driver/meshes/wheel_subassem.stl.stl scale=0.001 0.001 0.001
- added link steering_wheel_rl; visual mesh filename=package://driver/meshes/wheel_subassem.stl.stl scale=0.001 0.001 0.001
- added link steering_wheel_rr; visual mesh filename=package://driver/meshes/wheel_subassem.stl.stl scale=0.001 0.001 0.001
- link base_link: geometry visual mesh filename=package://driver/meshes/chassis-subassem.stl scale=0.001 0.001 0.001
Joints:
- added joint body_to_flw: type floating, parent base_link, child steering_wheel_fl, origin xyz=0 -0.22 0.25
- added joint body_to_frw: type floating, parent base_link, child steering_wheel_fr, origin xyz=0 -0.22 0.25
- added joint body_to_rlw: type floating, parent base_link, child steering_wheel_rl, origin xyz=0 -0.22 0.25
- added joint body_to_rrw: type floating, parent base_link, child steering_wheel_rr, origin xyz=0 -0.22 0.25
- added joint body_to_steering: type floating, parent base_link, child steering_subassem, origin xyz=0 -0.22 0.25
- added joint flw_to_steering: type floating, parent steering_subassem, child steering_wheel_fl, origin xyz=0 -0.22 0.25
- added joint frw_to_steering: type floating, parent steering_subassem, child steering_wheel_fr, origin xyz=0 -0.22 0.25

Commit message: steering wheel mesh added, steering visualization node implemented & tested

File: src/driver/urdf/robot.urdf (robot description, URDF)
Before this commit: robot Alan-v2, 6 links, 7 joints
Links:
- link steering_subassem: geometry visual mesh filename=package://driver/meshes/steering_subassem.stl scale=0.001 0.001 0.001
- link steering_wheel_fl: geometry visual mesh filename=package://driver/meshes/fl_wheel.stl scale=0.001 0.001 0.001
- link steering_wheel_fr: geometry visual mesh filename=package://driver/meshes/fr_wheel.stl scale=0.001 0.001 0.001
- link steering_wheel_rl: geometry visual mesh filename=package://driver/meshes/rl_wheel.stl scale=0.001 0.001 0.001
- link steering_wheel_rr: geometry visual mesh filename=package://driver/meshes/rr_wheel.stl scale=0.001 0.001 0.001
Joints:
- joint body_to_flw: origin xyz=0 -0.22 0.25 -> xyz=0 0 0; type floating -> continuous
- joint body_to_frw: origin xyz=0 -0.22 0.25 -> xyz=0 0 0; type floating -> continuous
- joint body_to_rlw: origin xyz=0 -0.22 0.25 -> xyz=0 0 0; type floating -> continuous
- joint body_to_rrw: origin xyz=0 -0.22 0.25 -> xyz=0 0 0; type floating -> continuous
- joint body_to_steering: origin xyz=0 -0.22 0.25 -> xyz=0 0 0; type floating -> fixed
- joint flw_to_steering: origin xyz=0 -0.22 0.25 -> xyz=0 0 0; type floating -> continuous
- joint frw_to_steering: origin xyz=0 -0.22 0.25 -> xyz=0 0 0; type floating -> continuous

Commit message: small changes to robot model. All packages created

File: src/driver/urdf/robot.urdf (robot description, URDF)
Before this commit: robot Alan-v2, 6 links, 7 joints
Joints:
- removed joint body_to_flw
- removed joint body_to_frw
- joint body_to_rrw: origin xyz=0 0 0 -> xyz=0.0 0 0

Commit message: steer train script changes & others

File: src/driver/urdf/robot.urdf (robot description, URDF)
Before this commit: robot Alan-v2, 6 links, 5 joints
Joints:
- joint body_to_rlw: type continuous -> fixed
- joint body_to_rrw: type continuous -> fixed
- joint flw_to_steering: type continuous -> fixed
- joint frw_to_steering: type continuous -> fixed

Commit message: begin training on new dataset

File: src/driver/urdf/robot.urdf (robot description, URDF)
Before this commit: robot Alan-v2, 6 links, 5 joints
Links:
- added link steering_col_subassem; visual mesh filename=package://driver/meshes/steering_col_subassem.stl scale=0.001 0.001 0.001
Joints:
- added joint body_to_steering_col: type fixed, parent base_link, child steering_col_subassem, origin xyz=0 0 0
